Commit message: modified scan match,and add time out protect and pose err control in client'

File: src/a_robot_platform/launch/orange_car.urdf (robot description, URDF)
Before this commit: robot OrangeCar, 3 links, 2 joints
Joints:
- joint laser_link_joint: origin xyz=0.1 0 0.28 rpy=0 0 3.1415926 -> xyz=0.1 0 0 rpy=0 0 3.1415926
